File: _saved_opensolar.sch (KiCad schematic (older format))
At the start: 136 parts, among them P1 USB_OTG, P2 microSD, P3 Panel+, P4 Panel-, P5 Batt-, P6 Batt+, Q1 IPP076N12N3, Q2 IPP076N12N3, Q3 IPP076N12N3, Q4 IPP076N12N3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

Commit message: recent chages and add docs
Parts:
- D1, D2, D3, D4, D5, D6: footprint (none) -> Diodes_SMD:D_SOD-123F
- L2: footprint (none) -> Inductors:PQ3218-3r3-70-t
- Q5, Q6: footprint (none) -> TO_SOT_Packages_SMD:SOT-23_Handsoldering
Changed lines of the file:
@@
 F 0 "L2" V 8450 1300 50  0000 L CNN
 F 1 "3.3uH  PQ3218-3R3-70-T" V 8350 750 50  0000 L CNN
-F 2 "" H 8400 1300 50  0001 C CNN
+F 2 "Inductors:PQ3218-3r3-70-t" H 8400 1300 50  0001 C CNN
 F 3 "" H 8400 1300 50  0000 C CNN
 	1    8400 1300
@@
 F 0 "D4" H 7750 5180 50  0000 L CNN
 F 1 "DFLS1100-7" H 7520 5020 50  0000 L CNN
-F 2 "" V 7800 5100 50  0001 C CNN
+F 2 "Diodes_SMD:D_SOD-123F" V 7800 5100 50  0001 C CNN
 F 3 "" V 7800 5100 50  0000 C CNN
 	1    7800 5100
@@
 F 0 "D1" H 1400 7550 50  0000 C CNN
 F 1 "D_Schottky" H 1400 7650 50  0000 C CNN
-F 2 "" H 1400 7450 50  0001 C CNN
+F 2 "Diodes_SMD:D_SOD-123F" H 1400 7450 50  0001 C CNN
 F 3 "" H 1400 7450 50  0000 C CNN
 	1    1400 7450
@@
 F 0 "Q6" H 3650 7275 50  0000 L CNN
 F 1 "S8050" H 3650 7200 50  0000 L CNN
-F 2 "" H 3650 7125 50  0001 L CIN
+F 2 "TO_SOT_Packages_SMD:SOT-23_Handsoldering" H 3650 7125 50  0001 L CIN
 F 3 "" H 3450 7200 50  0000 L CNN
 	1    3450 7200
@@
 F 0 "Q5" H 3050 7275 50  0000 L CNN
 F 1 "S8050" H 3050 7200 50  0000 L CNN
-F 2 "" H 3050 7125 50  0001 L CIN
+F 2 "TO_SOT_Packages_SMD:SOT-23_Handsoldering" H 3050 7125 50  0001 L CIN
 F 3 "" H 2850 7200 50  0000 L CNN
 	1    2850 7200
@@
 F 0 "D2" H 7350 1300 50  0000 C CNN
 F 1 "D_Schottky" H 7350 1100 50  0000 C CNN
-F 2 "" H 7350 1200 50  0001 C CNN
+F 2 "Diodes_SMD:D_SOD-123F" H 7350 1200 50  0001 C CNN
 F 3 "" H 7350 1200 50  0000 C CNN
 	1    7350 1200
@@
 F 0 "D3" H 7350 1900 50  0000 C CNN
 F 1 "D_Schottky" H 7350 1700 50  0000 C CNN
-F 2 "" H 7350 1800 50  0001 C CNN
+F 2 "Diodes_SMD:D_SOD-123F" H 7350 1800 50  0001 C CNN
 F 3 "" H 7350 1800 50  0000 C CNN
 	1    7350 1800
@@
 F 0 "D5" H 9500 1300 50  0000 C CNN
 F 1 "D_Schottky" H 9500 1100 50  0000 C CNN
-F 2 "" H 9500 1200 50  0001 C CNN
+F 2 "Diodes_SMD:D_SOD-123F" H 9500 1200 50  0001 C CNN
 F 3 "" H 9500 1200 50  0000 C CNN
 	1    9500 1200
@@
 F 0 "D6" H 9500 1900 50  0000 C CNN
 F 1 "D_Schottky" H 9500 1700 50  0000 C CNN
-F 2 "" H 9500 1800 50  0001 C CNN
+F 2 "Diodes_SMD:D_SOD-123F" H 9500 1800 50  0001 C CNN
 F 3 "" H 9500 1800 50  0000 C CNN
 	1    9500 1800
