File: opensolar.sch (KiCad schematic (older format))
At the start: 136 parts, among them P1 USB_OTG, P2 microSD, P3 Panel+, P4 Panel-, P5 Batt-, P6 Batt+, Q1 IPP076N12N3, Q2 IPP076N12N3, Q3 IPP076N12N3, Q4 IPP076N12N3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

Commit message: max5033
Parts:
- added C57: C, symbol C
- added C?: 0.1uf, symbol C
- added L?: 220uh, symbol INDUCTOR_SMALL
- added R? (x2): R, symbol R
- added U6: AZ1117H50, TO_SOT_Packages_SMD:SOT-223, symbol AP111750
- added U?: MAX5033, symbol MAX5033
- D1, D2, D3, D4, D5, D6: footprint (none) -> Diodes_SMD:D_SOD-123F
- L2: footprint (none) -> Inductors:PQ3218-3r3-70-t
- Q5, Q6: footprint (none) -> TO_SOT_Packages_SMD:SOT-23_Handsoldering
Connections:
- net +48V: now also R?.2
- net +5V: now also C57.1, U6.2 (VO), U6.4 (VO)
- net 10V: now also U6.3 (VI)
- net GND: now also C57.2, C?.2, R?.1, U6.1 (GND/ADJ), U?.3 (SGND), U?.6 (GND)
- new net: C?.1, U?.2 (VD)
- new net: R?.1, R?.2, U?.5 (ON)

Commit message: comments, enlarge sheet, footprints
Parts:
- added C59: 0.1uf 16v, Capacitors_SMD:C_0603_HandSoldering, symbol C
- added C60, C61: 33uf 10v, symbol CP
- added C62: 47uf 100v, symbol CP
- added D7: D_Schottky, Diodes_SMD:D_SOD-123F, symbol D_Schottky
- C57: value C -> 10uf 16v; footprint (none) -> Capacitors_SMD:C_0603_HandSoldering
- C58: renamed from C?; value 0.1uf -> 0.1uf 16v; footprint (none) -> Capacitors_SMD:C_0603_HandSoldering
- R48: renamed from R?; value R -> 10k; footprint (none) -> Resistors_SMD:R_0603_HandSoldering
- R49: renamed from R?; value R -> DNP; footprint (none) -> Resistors_SMD:R_0603_HandSoldering
- U1: footprint Resistors_SMD:R_0603_HandSoldering -> Housings_SOIC:SOIC-16_3.9x9.9mm_Pitch1.27mm
- U2: footprint (none) -> Housings_SSOP:TSSOP-28_4.4x9.7mm_Pitch0.65mm
- U4: footprint (none) -> SOIC127P1030X265-28N:SOIC127P1030X265-28N
- U5: footprint (none) -> SOP65P490X110-8N:SOP65P490X110-8N
- gave numbers to parts that had none: 2
Connections:
- net +3V3: now also L3.2, U7.4 (FB), C61.1
- net +48V: now also U7.7 (VIN), C62.1
- net +5V: now also C60.1; no longer C57.1
- net 10V: now also C57.1
- net GND: now also C60.2, C61.2, C62.2, D7.2 (A)
- net at U7.1 (BST): now also C59.2
- net at U7.8 (LX): now also L3.1, C59.1, D7.1 (K)
Other:
- note added: "100v absolute maximum open circuit input, \n48 volt lead acid battery (max 76 volts)\n50-65 amp limitation (to be tested)\nMPPT charge controller with wifi management\n"
- note added: "10V gate drive power supply\nOnly on during sunlight"
- note added: "3v3 @ 500mA\nAlways on\nPowered off batteries\nMax 76 volts input\nMin 7.5 volts input"
- note added: "Linear regulator\n10Vin--> 5Vout\nonly on during sunlight"
- note added: "Notes:\n-add on-board temp measurement for thermal shutdown\n-add external connector for battery thermocouple\n-connect thermocouple to esp ADC?\n-but ESP also needs ADC to measure battery voltage during no sunlight\n-evaluate replacements for SM72485 (possibly another MAX chip)\n-Voltage limits on input capacitors rather low. Alternative?\n-Can this be run without Panel Mode components?????\n-fi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"
- note added: "R49 and R48 can be voltage divided\nto set an undervoltage lock out\nVuvlo=(1+R48/R49)*1.85\nR48+R49<1M"
- note added: "possibly just use non polarized \n10uf cap if cost way less"
- note removed: "100v input, 48 volt lead acid battery max\n65 amp limitation\nMPPT charge controller with wifi management\n"
- moved on the sheet: C10, C35, C36, C37, C38, C5, C54, C58, C6, C8, D1, D4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
