File: opensolar.sch (KiCad schematic (older format))
At the start: 150 parts, among them P1 USB_OTG, P2 microSD, P3 Panel+, P4 Panel-, P5 Batt-, P6 Batt+, Q1 IPP076N12N3, Q2 IPP076N12N3, Q3 IPP076N12N3, Q4 IPP076N12N3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

Commit message: add temp sensing
Parts:
- added U?: SA56004X, MODULE, symbol SA56004X
- added W?: TP_D+, symbol TEST_1P
- added W?: TP_D-, symbol TEST_1P
- added W?: TP_CRIT, symbol TEST_1P
- added W?: TP_ALERT, symbol TEST_1P
Connections:
- net +3V3: now also U?.1 (VDD)
- net GND: now also U?.5 (GND)
- net SCL: now also U?.8 (SCLK)
- net SDA: now also U?.7 (SDATA)
- new net: U?.2 (D+), W?.1
- new net: U?.3 (D-), W?.1
- new net: U?.4 (T_CRIT), W?.1
- new net: U?.6 (ALERT), W?.1
Other:
- note added: "Notes:\n-add on-board temp measurement for thermal shutdown over I2C\n-add external connector for battery thermocouple\n-evaluate replacements for SM72485 (possibly another MAX chip)\n-Voltage limits on input capacitors rather low. Alternative?\n-Can this be run without Panel Mode components?????\n-find new shotkey diode with forward voltage drop under 0.45v\n"
- note removed: "Notes:\n-add on-board temp measurement for thermal shutdown\n-add external connector for battery thermocouple\n-connect thermocouple to esp ADC?\n-but ESP also needs ADC to measure battery voltage during no sunlight\n-evaluate replacements for SM72485 (possibly another MAX chip)\n-Voltage limits on input capacitors rather low. Alternative?\n-Can this be run without Panel Mode components?????\n-fi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"

Commit message: start layout
Parts:
- C60, C61: footprint (none) -> Capacitors_SMD:C_1206_HandSoldering
- C62: footprint (none) -> Capacitors_SMD:CP_Elec_10x10
- P1: footprint Connect:USB_Micro-B -> Connectors:USB_Micro-B
- Q1, Q2, Q3, Q4: footprint TO_SOT_Packages_THT:TO-220_Neutral123_Vertical -> TO_SOT_Packages_THT:TO-220_Vertical
- U8: renamed from U?; footprint MODULE -> Housings_SOIC:SOIC-8_3.9x4.9mm_Pitch1.27mm
- W1, W2, W3, W4, W5, W6: footprint Connect:1pin -> Connectors:PINTST
- W10, W11, W12, W7, W8, W9: renamed from W?; footprint (none) -> Connectors:PINTST
Other:
- note added: "Notes:\n-evaluate replacements for SM72485 (possibly another MAX chip)\n-Voltage limits on input capacitors rather low. Alternative?\n-Can this be run without Panel Mode components?????\n-find new shotkey diode with forward voltage drop under 0.45v\n"
- note removed: "Notes:\n-add on-board temp measurement for thermal shutdown over I2C\n-add external connector for battery thermocouple\n-evaluate replacements for SM72485 (possibly another MAX chip)\n-Voltage limits on input capacitors rather low. Alternative?\n-Can this be run without Panel Mode components?????\n-find new shotkey diode with forward voltage drop under 0.45v\n"
